File: Arduino Giga .kicad_sch (KiCad schematic)
At the start: 68 parts, among them IC10 PE4251MLI-Z, IC11 PE4251MLI-Z, IC3 ADG904BRUZ-REEL7, IC4 PE4251MLI-Z, IC8 PE4251MLI-Z, IC9 PE4251MLI-Z, J10 Conn_01x02, J11 RX1, J12 Conn_01x02, J4 Conn_01x02, J40 RX2, J41 Ringdown, J5 Digital, J6 Ringdown, J8 TX1, U1 SN74LV4052ADR, U2 Si5351A-B-GM, U4 LM4562MAX/NOPB, Y1 ABM8G-25.000MHZ-B4Y-T

Commit message: Arduino NMR 5.4: self-contained libraries, split BOMs, production release
Consolidate every footprint the design uses into Arduino_NMR.pretty so a
fresh clone resolves without the author's personal library table. Recover
L_0805_2012Metric_Pad1.15x1.40mm_HandSolder, dropped from KiCad 10's stock
library, from the board itself. Repoint 261 references and drop the dead
'Library' fp-lib-table entry.

Add tools/split_bom.py, which splits the board into JLCPCB assembly, back-side
hand solder, front-side hand solder and off-board parts, with matching
placement files. Chip packages are normalised to the short form (0402, 0805)
because the full KiCad name makes JLCPCB's matcher offer 01005 parts.

Add tools/check_selfcontained.py as a pre-push guard; it now passes 32/32.
Move six sheets not in the hierarchy to archive/. Prune two unused cached
symbols and three dead cached footprint defaults.

Co-Authored-By: Claude Opus 5 <noreply@anthropic.com>
Parts:
- removed C32, C42: 100 pF, Capacitor_SMD:C_0805_2012Metric_Pad1.18x1.45mm_HandSolder, symbol Device:C
- removed IC9: PE4251MLI-Z, Arduino:SOP65P490X106-9N, symbol PE:PE4251MLI-Z
- added C142, C143, C145, C146, C150, C151, C152, C153: 180 pF, Arduino_NMR:C_0805_2012Metric_Pad1.18x1.45mm_HandSolder, symbol Device:C
- added C148, C149, C154, C155, C63, C67, C68, C69: 47 pF, Arduino_NMR:C_0805_2012Metric_Pad1.18x1.45mm_HandSolder, symbol Device:C
- added J7: Conn_01x05, Arduino_NMR:PinHeader_1x05_P2.54mm_Vertical, symbol Connector_Generic:Conn_01x05
- added L14, L16, L17, L18, L48, L49, L52, L53: 330 nH, Arduino_NMR:L_0805_2012Metric_Pad1.05x1.20mm_HandSolder, symbol Device:L
- added L45, L46, L50, L51: 470 nH, Arduino_NMR:L_0805_2012Metric_Pad1.05x1.20mm_HandSolder, symbol Device:L
- added R18: 50Ω, Arduino_NMR:R_0805_2012Metric_Pad1.20x1.40mm_HandSolder, symbol Device:R_US
- AT2: footprint Arduino:PE43711B-Z -> Arduino_NMR:PE43711B-Z
- C1, C14, C15, C16, C2, C27, C28, C29, C3, C33, C39, C4, C5, C6, C8, C9: footprint Capacitor_SMD:C_0805_2012Metric_Pad1.18x1.45mm_HandSolder -> Arduino_NMR:C_0805_2012Metric
- C10, C141, C144, C147, C17, C18, C19, C24, C62: footprint Capacitor_SMD:C_0805_2012Metric_Pad1.18x1.45mm_HandSolder -> Arduino_NMR:C_0805_2012Metric; now in the parts list
- C43: value 1 pF -> 100 nF; footprint Capacitor_SMD:C_0805_2012Metric_Pad1.18x1.45mm_HandSolder -> Arduino_NMR:C_0805_2012Metric
- D1: footprint Diode_SMD:D_SMA_Handsoldering -> Arduino_NMR:D_SMA_Handsoldering; now in the parts list
- IC10, IC11, IC4, IC8: footprint Arduino:SOP65P490X106-9N -> Arduino_NMR:SOP65P490X106-9N
- IC3: footprint Imported:ADG904BRUZ -> Arduino_NMR:ADG904BRUZ
- J10, J12, J4: footprint Connector_PinHeader_2.54mm:PinHeader_1x02_P2.54mm_Vertical -> Arduino_NMR:PinHeader_1x02_P2.54mm_Vertical; now in the parts list
- J11, J40, J41, J6, J8: footprint Connector_Coaxial:SMA_Amphenol_901-144_Vertical -> Arduino_NMR:SMA_Amphenol_901-144_Vertical; now in the parts list
- J5: footprint Connector_PinHeader_2.54mm:PinHeader_2x18_P2.54mm_Vertical -> Arduino_NMR:PinHeader_2x18_P2.54mm_Vertical; now in the parts list
- JP2, JP5, JP8: footprint Jumper:SolderJumper-2_P1.3mm_Open_Pad1.0x1.5mm -> Arduino_NMR:SolderJumper-2_P1.3mm_Open_Pad1.0x1.5mm; now in the parts list
- JP4: footprint Jumper:SolderJumper-3_P1.3mm_Open_Pad1.0x1.5mm -> Arduino_NMR:SolderJumper-3_P1.3mm_Open_Pad1.0x1.5mm; now in the parts list
- L13, L44, L47: footprint Inductor_SMD:L_0805_2012Metric_Pad1.15x1.40mm_HandSolder -> Arduino_NMR:L_0805_2012Metric_Pad1.15x1.40mm_HandSolder; now in the parts list
- R1, R10, R13, R14, R15, R3, R4, R6, R7, R9: footprint Resistor_SMD:R_0805_2012Metric_Pad1.20x1.40mm_HandSolder -> Arduino_NMR:R_0805_2012Metric_Pad1.20x1.40mm_HandSolder
- R5, R8: footprint Resistor_SMD:R_0805_2012Metric_Pad1.20x1.40mm_HandSolder -> Arduino_NMR:R_0805_2012Metric_Pad1.20x1.40mm_HandSolder; LCSC Part # (none) -> 0805W8F1001T5E
- U1: footprint Package_SO:SOIC-16_3.9x9.9mm_P1.27mm -> Arduino_NMR:SOIC-16_3.9x9.9mm_P1.27mm
- U2: footprint Package_DFN_QFN:QFN-20-1EP_4x4mm_P0.5mm_EP2.7x2.7mm -> Arduino_NMR:QFN-20-1EP_4x4mm_P0.5mm_EP2.7x2.7mm
- U4: footprint Imported:SOIC-8-1EP_3.9x4.9mm_P1.27mm_EP2.29x3mm_nobottomgnd -> Arduino_NMR:SOIC-8-1EP_3.9x4.9mm_P1.27mm_EP2.29x3mm_nobottomgnd
- Y1: footprint Crystal:Crystal_SMD_SeikoEpson_FA238-4Pin_3.2x2.5mm_HandSoldering -> Arduino_NMR:Crystal_SMD_SeikoEpson_FA238-4Pin_3.2x2.5mm_HandSoldering
Connections:
- net +5V is gone; now on net +3V3: C3.1, U1.16 (VCC)
- net Demod_B is gone; now on net CLK_4_QB: U1.9 (B_90)
- net Atten: now also AT2.14 (RF2), IC8.3 (RFC); no longer AT2.5 (RF1), IC8.5 (RF1)
- net CTL_5V (PI10): no longer J5.14 (Pin_14)
- net CTL_MUX (PK5): no longer J5.21 (Pin_21)
- net CTL_RFIN (PK2): now also C29.2, IC8.2 (V1)
- net CTL_TX_or_DEMOD (PK7): no longer C29.2, IC8.2 (V1), J5.16 (Pin_16)
- net GND: now also U1.6 (INH), C142.1, C143.1, C145.1, C146.1, C148.1, C149.1, C150.1, C151.1, C152.1, C153.1, C154.1, C155.1, C63.1, C67.1, C68.1, C69.1, R18.2
- net RX_A: now also C154.2, L52.1; no longer J11.1 (In)
- net RX_B: now also C155.2, L53.1; no longer J40.1 (In)
- net TX_A: now also C148.2, L48.1; no longer J8.1 (In)
- net TX_B: now also C149.2, L49.1; no longer J6.1 (In)
- net TX_SWITCH: now also IC8.8 (RF2); no longer AT2.14 (RF2)
- net +12V renamed +9V_SYS
- net Attem_Demod renamed SW_To_Demod
- net SW_To_Demod: now also AT2.5 (RF1); no longer IC8.3 (RFC)
- net CLK_4_QA renamed CLK_4_QB
- net CLK_5_QB renamed CLK_5_QA
- net CLK_5_QA: now also U1.10 (A_0)
- removed net Demod_A: IC8.8 (RF2), U1.10 (A_0)
- new net: C142.2, L14.1, L45.2
- new net: C63.2, J8.1 (In), L14.2
- new net: C151.2, L18.1, L51.2
- new net: C69.2, J40.1 (In), L18.2
- new net: C146.2, L46.1, L49.2
- new net: C143.2, L16.1, L46.2
- new net: C68.2, J11.1 (In), L17.2
- new net: IC8.5 (RF1), R18.1
- new net: C150.2, L17.1, L50.2
- new net: C152.2, L50.1, L52.2
- new net: C153.2, L51.1, L53.2
- new net: C145.2, L45.1, L48.2
- new net: C67.2, J6.1 (In), L16.2
- new net PI10: J5.14 (Pin_14)
- new net PK5: J5.21 (Pin_21)
- new net PK7: J5.16 (Pin_16)
- new net TTL1: J7.1 (Pin_1)
- new net TTL2: J7.2 (Pin_2)
- new net TTL3: J7.3 (Pin_3)
- new net TTL4: J7.4 (Pin_4)
- new net TTL5: J7.5 (Pin_5)
Other:
- note removed: "Controls the multiplexer (MUX) frequency between PLLA and PLLB."
- moved on the sheet: C27, C28, C29, D1, IC4, IC8, J11, J40, J41, J6, J8, JP2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
