File: Arduino_NMR_5.4.kicad_sch (KiCad schematic)
At the start: 3 parts, among them J16 RFShield_OnePiece, J17 RFShield_OnePiece, J32 RFShield_OnePiece

Commit message: Arduino NMR 5.4: self-contained libraries, split BOMs, production release
Consolidate every footprint the design uses into Arduino_NMR.pretty so a
fresh clone resolves without the author's personal library table. Recover
L_0805_2012Metric_Pad1.15x1.40mm_HandSolder, dropped from KiCad 10's stock
library, from the board itself. Repoint 261 references and drop the dead
'Library' fp-lib-table entry.

Add tools/split_bom.py, which splits the board into JLCPCB assembly, back-side
hand solder, front-side hand solder and off-board parts, with matching
placement files. Chip packages are normalised to the short form (0402, 0805)
because the full KiCad name makes JLCPCB's matcher offer 01005 parts.

Add tools/check_selfcontained.py as a pre-push guard; it now passes 32/32.
Move six sheets not in the hierarchy to archive/. Prune two unused cached
symbols and three dead cached footprint defaults.

Co-Authored-By: Claude Opus 5 <noreply@anthropic.com>
Parts:
- J16: footprint Arduino:RF Shield_1 -> Arduino_NMR:RF Shield_1; now in the parts list
- J17: footprint Arduino:RF Shield_3 -> Arduino_NMR:RF Shield_3; now in the parts list
- J32: footprint Arduino:RF Shield_2 -> Arduino_NMR:RF Shield_2; now in the parts list
Connections:
- net GND: no longer J16.1 (Shield)
Changed lines of the file:
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@@
 		)
 		(instances
-			(project "Arduino_NMR_5.2"
+			(project "Arduino_NMR_5.4"
 				(path "/e63e39d7-6ac0-4ffd-8aa3-1841a4541b55"
 					(reference "#PWR0133")
@@
 		)
 		(instances
-			(project "Arduino_NMR_5.2"
+			(project "Arduino_NMR_5.4"
 				(path "/e63e39d7-6ac0-4ffd-8aa3-1841a4541b55"
 					(reference "#PWR0131")
@@
 		(body_style 1)
 		(exclude_from_sim no)
-		(in_bom no)
+		(in_bom yes)
 		(on_board yes)
 		(in_pos_files no)
@@
 			)
 		)
-		(property "Footprint" "Arduino:RF Shield_2"
+		(property "Footprint" "Arduino_NMR:RF Shield_2"
 			(at 87.63 26.67 0)
 			(hide yes)
@@
 		)
 		(instances
-			(project "Arduino_NMR_5.2"
+			(project "Arduino_NMR_5.4"
 				(path "/e63e39d7-6ac0-4ffd-8aa3-1841a4541b55"
 					(reference "J32")
@@
 		(body_style 1)
 		(exclude_from_sim no)
-		(in_bom no)
+		(in_bom yes)
 		(on_board yes)
 		(in_pos_files no)
@@
 			)
 		)
-		(property "Footprint" "Arduino:RF Shield_3"
+		(property "Footprint" "Arduino_NMR:RF Shield_3"
 			(at 140.97 26.67 0)
 			(hide yes)
@@
 		)
 		(instances
-			(project "Arduino_NMR_5.2"
+			(project "Arduino_NMR_5.4"
 				(path "/e63e39d7-6ac0-4ffd-8aa3-1841a4541b55"
 					(reference "J17")
@@
 		)
 		(instances
-			(project "Arduino_NMR_5.2"
+			(project "Arduino_NMR_5.4"
 				(path "/e63e39d7-6ac0-4ffd-8aa3-1841a4541b55"
 					(reference "#PWR035")
@@
 		(body_style 1)
 		(exclude_from_sim no)
-		(in_bom no)
+		(in_bom yes)
 		(on_board yes)
 		(in_pos_files no)
@@
 			)
 		)
-		(property "Footprint" "Arduino:RF Shield_1"
+		(property "Footprint" "Arduino_NMR:RF Shield_1"
 			(at 36.83 25.4 0)
 			(hide yes)
@@
 		)
 		(instances
-			(project "Arduino_NMR_5.2"
+			(project "Arduino_NMR_5.4"
 				(path "/e63e39d7-6ac0-4ffd-8aa3-1841a4541b55"
 					(reference "J16")
@@
 		)
 		(instances
-			(project "Arduino_NMR_5.2"
+			(project "Arduino_NMR_5.4"
 				(path "/e63e39d7-6ac0-4ffd-8aa3-1841a4541b55"
 					(page "4")
@@
 		)
 		(instances
-			(project "Arduino_NMR_5.2"
+			(project "Arduino_NMR_5.4"
 				(path "/e63e39d7-6ac0-4ffd-8aa3-1841a4541b55"
 					(page "7")
@@
 		)
 		(instances
-			(project "Arduino_NMR_5.2"
-				(path "/e63e39d7-6ac0-4ffd-8aa3-1841a4541b55"
-					(page "7")
-				)
-			)
+			(project "Arduino_NMR_5.4"
+				(path "/e63e39d7-6ac0-4ffd-8aa3-1841a4541b55"
+					(page "2")
+				)
+			)
