File: PHA_13HLN.kicad_sch (KiCad schematic)
At the start: 21 parts, among them IC13 PHA-13HLN+, IC14 PHA-13HLN+

Commit message: Arduino NMR 5.4: self-contained libraries, split BOMs, production release
Consolidate every footprint the design uses into Arduino_NMR.pretty so a
fresh clone resolves without the author's personal library table. Recover
L_0805_2012Metric_Pad1.15x1.40mm_HandSolder, dropped from KiCad 10's stock
library, from the board itself. Repoint 261 references and drop the dead
'Library' fp-lib-table entry.

Add tools/split_bom.py, which splits the board into JLCPCB assembly, back-side
hand solder, front-side hand solder and off-board parts, with matching
placement files. Chip packages are normalised to the short form (0402, 0805)
because the full KiCad name makes JLCPCB's matcher offer 01005 parts.

Add tools/check_selfcontained.py as a pre-push guard; it now passes 32/32.
Move six sheets not in the hierarchy to archive/. Prune two unused cached
symbols and three dead cached footprint defaults.

Co-Authored-By: Claude Opus 5 <noreply@anthropic.com>
Parts:
- C20, C46: footprint Capacitor_SMD:C_0402_1005Metric -> Arduino_NMR:C_0402_1005Metric; LCSC Part # (none) -> 0402CG1R5C500NT
- C30, C45, C60, C66: footprint Capacitor_SMD:C_0603_1608Metric -> Arduino_NMR:C_0603_1608Metric
- C31, C61: footprint Capacitor_SMD:C_0402_1005Metric -> Arduino_NMR:C_0402_1005Metric; LCSC Part # (none) -> CL05B104KO5NNNC
- C40, C64: footprint Capacitor_SMD:C_0402_1005Metric -> Arduino_NMR:C_0402_1005Metric; LCSC Part # (none) -> 0402B102K500NT
- C41, C65: footprint Capacitor_SMD:C_0805_2012Metric_Pad1.18x1.45mm_HandSolder -> Arduino_NMR:C_0805_2012Metric; LCSC Part # (none) -> GRM21BR61H106KE43L
- C47: footprint Capacitor_THT:C_Radial_D5.0mm_H5.0mm_P2.00mm -> Arduino_NMR:C_Radial_D5.0mm_H5.0mm_P2.00mm
- IC13, IC14: footprint imported:PHA13HLN -> Arduino_NMR:PHA13HLN
- L1, L3: footprint Inductor_SMD:L_0603_1608Metric -> Arduino_NMR:L_0603_1608Metric
- L15, L2: footprint Inductor_SMD:L_1210_3225Metric_Pad1.42x2.65mm_HandSolder -> Arduino_NMR:L_1210_3225Metric_Pad1.42x2.65mm_HandSolder
- R16, R17: footprint Resistor_SMD:R_0402_1005Metric_Pad0.72x0.64mm_HandSolder -> Arduino_NMR:R_0402_1005Metric_Pad0.72x0.64mm_HandSolder; LCSC Part # (none) -> 0402WGF1501TCE
