File: amp_power.kicad_sch (KiCad schematic)
At the start: 16 parts, among them IC1 SN74LV1T04DBVR, IC12 SN74LV1T04DBVR, IC2 SN74LV1T04DBVR, IC25 BD33GA5WEFJ-E2, IC5 TLV74125PDBVR, IC6 BD50GC0VEFJ-ME2, IC7 BD80GC0VEFJ-ME2, J1 PJ-058B

Commit message: Arduino NMR 5.4: self-contained libraries, split BOMs, production release
Consolidate every footprint the design uses into Arduino_NMR.pretty so a
fresh clone resolves without the author's personal library table. Recover
L_0805_2012Metric_Pad1.15x1.40mm_HandSolder, dropped from KiCad 10's stock
library, from the board itself. Repoint 261 references and drop the dead
'Library' fp-lib-table entry.

Add tools/split_bom.py, which splits the board into JLCPCB assembly, back-side
hand solder, front-side hand solder and off-board parts, with matching
placement files. Chip packages are normalised to the short form (0402, 0805)
because the full KiCad name makes JLCPCB's matcher offer 01005 parts.

Add tools/check_selfcontained.py as a pre-push guard; it now passes 32/32.
Move six sheets not in the hierarchy to archive/. Prune two unused cached
symbols and three dead cached footprint defaults.

Co-Authored-By: Claude Opus 5 <noreply@anthropic.com>
Parts:
- removed C11, C12, C21, C22, C23, C26: 10 nF, Capacitor_SMD:C_0805_2012Metric_Pad1.18x1.45mm_HandSolder, symbol Device:C
- removed IC25: BD33GA5WEFJ-E2, Arduino:SOIC127P600X100-9N, symbol BD80GC0MEFJ-ME2:BD80GC0MEFJ-ME2
- removed IC6: BD50GC0VEFJ-ME2, Arduino:SOIC127P600X100-9N, symbol BD80GC0MEFJ-ME2:BD80GC0MEFJ-ME2
- removed IC7: BD80GC0VEFJ-ME2, Arduino:SOIC127P600X100-9N, symbol BD80GC0MEFJ-ME2:BD80GC0MEFJ-ME2
- removed J1: PJ-058B, Arduino:PJ058B, symbol Arduino:PJ-058B
- added J2: Conn_01x12, Arduino_NMR:PinHeader_1x12_P2.54mm_Vertical, symbol Connector_Generic:Conn_01x12
- C34, C48: footprint Capacitor_SMD:C_0805_2012Metric_Pad1.18x1.45mm_HandSolder -> Arduino_NMR:C_0805_2012Metric; now in the parts list
- IC1, IC12, IC2: footprint Arduino:SOT95P280X145-5N -> Arduino_NMR:SOT95P280X145-5N
- IC5: footprint SOT95P280X145-5N -> Arduino_NMR:SOT95P280X145-5N
Connections:
- net +3V3: now also J2.4 (Pin_4)
- net +8V: now also J2.3 (Pin_3)
- net CTL_3V3 (PI13): now also J2.5 (Pin_5)
- net CTL_8V (PI14): now also J2.6 (Pin_6)
- new net +9V_SYS: J2.1 (Pin_1)
- new net TTL1: J2.8 (Pin_8)
- new net TTL2: J2.9 (Pin_9)
- new net TTL3: J2.10 (Pin_10)
- new net TTL4: J2.11 (Pin_11)
- new net TTL5: J2.12 (Pin_12)
Other:
- moved on the sheet: C34, C48
